File: PCB/led-matrix.kicad_pcb (KiCad board)
At the start: 2 copper layers, 10 parts

Commit message: Layout schematic
Parts:
- added C1: 100n, Capacitor_SMD:C_0603_1608Metric, F.Cu at (103.7, 63.1)
- added C10: 100n, Capacitor_SMD:C_0603_1608Metric, F.Cu at (107.7, 73.1)
- added C2: 100n, Capacitor_SMD:C_0603_1608Metric, F.Cu at (103.7, 65.6)
- added C3: 100n, Capacitor_SMD:C_0603_1608Metric, F.Cu at (103.7, 68.1)
- added C4: 100n, Capacitor_SMD:C_0603_1608Metric, F.Cu at (103.7, 70.6)
- added C5: 100n, Capacitor_SMD:C_0603_1608Metric, F.Cu at (103.7, 73.1)
- added C6: 100n, Capacitor_SMD:C_0603_1608Metric, F.Cu at (107.7, 63.1)
- added C7: 100n, Capacitor_SMD:C_0603_1608Metric, F.Cu at (107.7, 65.6)
- added C8: 100n, Capacitor_SMD:C_0603_1608Metric, F.Cu at (107.7, 68.1)
- added C9: 100n, Capacitor_SMD:C_0603_1608Metric, F.Cu at (107.7, 70.6)
- added J1: Conn_02x03_Odd_Even, Connector_PinHeader_2.54mm:PinHeader_2x03_P2.54mm_Vertical_SMD, F.Cu at (95.3, 66.7)
- moved D10 84.2 mm to (117.7, 58.4)
- moved D2 84.2 mm to (98.4, 51.7)
- moved D3 84.2 mm to (104.9, 51.7)
- moved D5 84.2 mm to (117.7, 51.7)
- moved D7 84.2 mm to (98.4, 58.4)
- moved D8 84.2 mm to (104.9, 58.4)
- moved D1 84.2 mm to (92.0, 51.7)
- moved D4 84.2 mm to (111.3, 51.7)
- moved D6 84.2 mm to (92.0, 58.4)
- moved D9 84.2 mm to (111.3, 58.4)
Connections:
- D1 pad 1: unconnected-(D1-DO-Pad1) -> Net-(D1-DO)
- D1 pad 2: unconnected-(D1-GND-Pad2) -> GND
- D1 pad 3: unconnected-(D1-VDD-Pad3) -> 5V
- D1 pad 4: unconnected-(D1-DI-Pad4) -> DIN
- D10 pad 1: unconnected-(D10-DO-Pad1) -> DOUT
- D10 pad 2: unconnected-(D10-GND-Pad2) -> GND
- D10 pad 3: unconnected-(D10-VDD-Pad3) -> 5V
- D10 pad 4: unconnected-(D10-DI-Pad4) -> Net-(D10-DI)
- D2 pad 1: unconnected-(D2-DO-Pad1) -> Net-(D2-DO)
- D2 pad 2: unconnected-(D2-GND-Pad2) -> GND
- D2 pad 3: unconnected-(D2-VDD-Pad3) -> 5V
- D2 pad 4: unconnected-(D2-DI-Pad4) -> Net-(D1-DO)
- D3 pad 1: unconnected-(D3-DO-Pad1) -> Net-(D3-DO)
- D3 pad 2: unconnected-(D3-GND-Pad2) -> GND
- D3 pad 3: unconnected-(D3-VDD-Pad3) -> 5V
- D3 pad 4: unconnected-(D3-DI-Pad4) -> Net-(D2-DO)
- D4 pad 2: unconnected-(D4-GND-Pad2) -> GND
- D4 pad 3: unconnected-(D4-VDD-Pad3) -> 5V
- D4 pad 4: unconnected-(D4-DI-Pad4) -> Net-(D3-DO)
- D5 pad 2: unconnected-(D5-GND-Pad2) -> GND
- D5 pad 3: unconnected-(D5-VDD-Pad3) -> 5V
- D6 pad 2: unconnected-(D6-GND-Pad2) -> GND
- D6 pad 3: unconnected-(D6-VDD-Pad3) -> 5V
- D7 pad 1: unconnected-(D7-DO-Pad1) -> Net-(D7-DO)
- D7 pad 2: unconnected-(D7-GND-Pad2) -> GND
- D7 pad 3: unconnected-(D7-VDD-Pad3) -> 5V
- D8 pad 1: unconnected-(D8-DO-Pad1) -> Net-(D8-DO)
- D8 pad 2: unconnected-(D8-GND-Pad2) -> GND
- D8 pad 3: unconnected-(D8-VDD-Pad3) -> 5V
- D8 pad 4: unconnected-(D8-DI-Pad4) -> Net-(D7-DO)
- D9 pad 1: unconnected-(D9-DO-Pad1) -> Net-(D10-DI)
- D9 pad 2: unconnected-(D9-GND-Pad2) -> GND
- D9 pad 3: unconnected-(D9-VDD-Pad3) -> 5V
- D9 pad 4: unconnected-(D9-DI-Pad4) -> Net-(D8-DO)

Commit message: Layout board
Parts:
- added C11: 100n, Capacitor_SMD:C_0603_1608Metric, B.Cu at (118.4, 70.8)
- added C12: 100n, Capacitor_SMD:C_0603_1608Metric, B.Cu at (128.4, 70.8)
- added D11: APA-106-F5, WS2812D:WS2812D, F.Cu at (118.4, 68.5)
- added D12: APA-106-F5, WS2812D:WS2812D, F.Cu at (128.4, 68.5)
- C1, C10, C2, C3, C4, C5, C6, C7, C8, C9, J1: moved to B.Cu
- moved D6 36.4 mm to (128.4, 58.5), turned to 180 degrees
- moved C7 29.8 mm to (78.4, 70.8)
- moved C1 26.2 mm to (78.4, 56.2)
- moved D7 22.4 mm to (78.4, 68.5), turned to 180 degrees
- moved C5 22.4 mm to (118.4, 56.2)
- moved C6 21.8 mm to (128.4, 56.2)
- moved C8 19.5 mm to (88.4, 70.8)
- moved D8 19.3 mm to (88.4, 68.5), turned to 180 degrees
- moved C2 17.9 mm to (88.4, 56.2)
- moved D9 16.4 mm to (98.4, 68.5), turned to 180 degrees
- moved D1 15.2 mm to (78.4, 58.5), turned to 180 degrees
- moved C4 15.1 mm to (108.4, 56.2)
- moved D10 13.7 mm to (108.4, 68.5), turned to 180 degrees
- moved C3 13.0 mm to (98.4, 56.2)
- moved D2 12.1 mm to (88.4, 58.5), turned to 180 degrees
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Connections:
- D10 pad 1: DOUT -> Net-(D10-DO)
- D4 pad 1: unconnected-(D4-DO-Pad1) -> Net-(D4-DO)
- D5 pad 1: unconnected-(D5-DO-Pad1) -> Net-(D5-DO)
- D5 pad 4: unconnected-(D5-DI-Pad4) -> Net-(D4-DO)
- D6 pad 1: unconnected-(D6-DO-Pad1) -> Net-(D6-DO)
- D6 pad 4: unconnected-(D6-DI-Pad4) -> Net-(D5-DO)
- D7 pad 4: unconnected-(D7-DI-Pad4) -> Net-(D6-DO)
Routing:
- net Net-(D6-DO): track 0.00 -> 59.2 mm
- net 5V: track 0.00 -> 37.5 mm, vias 0 -> 2
- net DOUT: track 0.00 -> 27.8 mm
- net DIN: track 0.00 -> 25.6 mm
- net Net-(D8-DO): track 0.00 -> 6.19 mm
- net Net-(D7-DO): track 0.00 -> 6.19 mm
- net Net-(D5-DO): track 0.00 -> 6.19 mm
- net Net-(D4-DO): track 0.00 -> 6.19 mm
- net Net-(D3-DO): track 0.00 -> 6.19 mm
- net Net-(D2-DO): track 0.00 -> 6.19 mm
- net Net-(D11-DO): track 0.00 -> 6.19 mm
- net Net-(D10-DO): track 0.00 -> 6.19 mm
- net Net-(D10-DI): track 0.00 -> 6.19 mm
- net Net-(D1-DO): track 0.00 -> 6.19 mm
- net GND: track 0.00 -> 5.05 mm
- added copper zone on F.Cu, net 5V
- added copper zone on B.Cu, net GND
Other:
- board outline added: 58 x 18 mm

Commit message: Rearrange board layout
Parts:
- moved C3 2.83 mm to (95.5, 56.2), turned to 180 degrees
- moved C10 1.99 mm to (110.3, 70.8)
- moved C4 1.90 mm to (110.3, 56.3)
- moved C9 1.78 mm to (96.5, 70.8), turned to 180 degrees
- turned D10 to -135 degrees
- turned D3 to -135 degrees
- turned D4 to 135 degrees
- turned D9 to 135 degrees
Routing:
- net 5V: track 37.5 -> 40.0 mm
- net Net-(D6-DO): track 59.2 -> 61.5 mm
- net DIN: track 25.6 -> 27.2 mm
- net DOUT: track 27.8 -> 29.0 mm
- net Net-(D3-DO): track 6.19 -> 7.31 mm
- net Net-(D10-DI): track 6.19 -> 7.31 mm
- net Net-(D8-DO): track 6.19 -> 7.31 mm
- net Net-(D4-DO): track 6.19 -> 7.31 mm
- net Net-(D2-DO): track 6.19 -> 7.31 mm
- net Net-(D10-DO): track 6.19 -> 7.31 mm

Commit message: Add bill of materials
Other:
- board text added: "ImSeanConroy/LED-Matrix (v0.1)"
Changed lines of the file:
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@@
 		(tags "capacitor")
 		(property "Reference" "C9"
-			(at 0 1.43 360)
+			(at 0 1.43 0)
 			(layer "B.SilkS")
 			(hide yes)
@@
 		)
 		(property "Value" "100n"
-			(at 0 -1.43 360)
+			(at 0 -1.43 0)
 			(layer "B.Fab")
 			(hide yes)
@@
 		)
 		(fp_text user "${REFERENCE}"
-			(at 0 0 360)
+			(at 0 0 0)
 			(layer "B.Fab")
 			(effects
@@
 		(tags "capacitor")
 		(property "Reference" "C3"
-			(at 0 1.43 360)
+			(at 0 1.43 0)
 			(layer "B.SilkS")
 			(hide yes)
@@
 		)
 		(property "Value" "100n"
-			(at 0 -1.43 360)
+			(at 0 -1.43 0)
 			(layer "B.Fab")
 			(hide yes)
@@
 		)
 		(fp_text user "${REFERENCE}"
-			(at 0 0 360)
+			(at 0 0 0)
 			(layer "B.Fab")
 			(effects
@@
 		(layer "Edge.Cuts")
 	)
+	(gr_text "ImSeanConroy/LED-Matrix (v0.1)"
+		(at 97.8 64.45 0)
+		(layer "B.SilkS")
+		(effects
+			(font
+				(size 0.85 0.85)
+				(thickness 0.1)
+			)
+			(justify left bottom mirror)
+		)
+	)
 	(via
