File: PCB/led-matrix.kicad_sch (KiCad schematic)
At the start: 10 parts

Commit message: Layout schematic
Parts:
- added C1, C10, C2, C3, C4, C5, C6, C7, C8, C9: 100n, Capacitor_SMD:C_0603_1608Metric, symbol Device:C_Small
- added J1: Conn_02x03_Odd_Even, Connector_PinHeader_2.54mm:PinHeader_2x03_P2.54mm_Vertical_SMD, symbol Connector_Generic:Conn_02x03_Odd_Even
Connections:
- net at D5.1 (DO): now also D6.4 (DI)
- net GND: now reaches D5.2 (GND)
- net GND: now also D1.2 (GND), D10.2 (GND), D2.2 (GND), D3.2 (GND), D4.2 (GND), D6.2 (GND), D7.2 (GND), D8.2 (GND), D9.2 (GND), C1.2, C10.2, C2.2, C3.2, C4.2, C5.2, C6.2, C7.2, C8.2, C9.2, J1.3 (Pin_3), J1.4 (Pin_4)
- net 5V: now reaches D5.3 (VDD)
- net 5V: now also D1.3 (VDD), D10.3 (VDD), D2.3 (VDD), D3.3 (VDD), D4.3 (VDD), D6.3 (VDD), D7.3 (VDD), D8.3 (VDD), D9.3 (VDD), C1.1, C10.1, C2.1, C3.1, C4.1, C5.1, C6.1, C7.1, C8.1, C9.1, J1.1 (Pin_1), J1.2 (Pin_2)
- net at D5.4 (DI): now also D4.1 (DO)
- net at D9.1 (DO): now also D10.4 (DI)
- net at D9.4 (DI): now also D8.1 (DO)
- net at D3.1 (DO): now also D4.4 (DI)
- net at D3.4 (DI): now also D2.1 (DO)
- net at D6.1 (DO): now also D7.4 (DI)
- net DOUT: now reaches D10.1 (DO)
- net DOUT: now also J1.6 (Pin_6)
- net at D1.1 (DO): now also D2.4 (DI)
- net DIN: now reaches D1.4 (DI)
- net DIN: now also J1.5 (Pin_5)
- net at D8.4 (DI): now also D7.1 (DO)
Other:
- moved on the sheet: D1, D10, D2, D3, D4, D5, D6, D7, D8, D9

Commit message: Layout board
Parts:
- added C11, C12: 100n, Capacitor_SMD:C_0603_1608Metric, symbol Device:C_Small
- added D11, D12: APA-106-F5, WS2812D:WS2812D, symbol LED:APA-106-F5
Connections:
- net 5V: now also C11.1, C12.1, D11.3 (VDD), D12.3 (VDD)
- net DOUT: now also D12.1 (DO); no longer D10.1 (DO)
- net GND: now also C11.2, C12.2, D11.2 (GND), D12.2 (GND)
- new net: D11.1 (DO), D12.4 (DI)
- new net: D10.1 (DO), D11.4 (DI)
Other:
- moved on the sheet: C1, C10, C2, C3, C4, C5, C6, C7, C8, C9, D1, D2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

Commit message: Resolve ground plane island issue
Other:
- title: (none) -> LED Matrix
Changed lines of the file:
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@@
 	(generator_version "8.0")
 	(paper "A4")
+	(title_block
+		(title "LED Matrix")
+		(date "2025-07-13")
+		(rev "0.2")
+	)
 	(junction
 		(at 215.9 111.76)
